Commit message: Gazebo Sim

File: description/robot.urdf.xacro (robot description, xacro)
@@ -5,3 +5,4 @@
     <xacro:include filename="inertial_macro.xacro"/>
     <xacro:include filename="robot_core.xacro"/>
+    <xacro:include filename="gazebo_control.xacro"/>
 </robot>

File: description/robot_core.xacro (robot description, xacro)
@@ -27,4 +27,7 @@
         </xacro:inertial_box>
     </link>
+    <gazebo reference="chassis">
+        <material>Gazebo/White</material>
+    </gazebo>
 <!-- left wheel joint -->
     <joint name="left_wheel_joint" type="continuous">
@@ -51,4 +54,7 @@
         </xacro:inertial_cylinder>
     </link>
+    <gazebo reference="left_wheel">
+        <material>Gazebo/Blue</material>
+    </gazebo>
     <!-- right wheel joint -->
     <joint name="right_wheel_joint" type="continuous">
@@ -75,4 +81,7 @@
         </xacro:inertial_cylinder>
     </link>
+    <gazebo reference="right_wheel">
+        <material>Gazebo/Blue</material>
+    </gazebo>
     <!-- caster wheel joint -->
     <joint name="caster_wheel_joint" type="fixed">
@@ -98,3 +107,8 @@
         </xacro:inertial_sphere>
     </link>
+    <gazebo reference="caster_wheel">
+        <material>Gazebo/Black</material>
+        <mu1 value = "0.001" />
+        <mu2 value = "0.001" />
+    </gazebo>
 </robot>
