Commit message: ros2_controller_test_with_errors

File: description/lidar.xacro (robot description, xacro)
@@ -47,5 +47,5 @@
             <plugin name="laser_controller" filename="libgazebo_ros_ray_sensor.so">
                 <ros>
-                    <argument>~/out:=scan</argument>
+                    <argument>--ros-args --remap ~/out:=scan</argument>
                 </ros>
                 <output_type>sensor_msgs/LaserScan</output_type>

File: description/properties.xacro (robot description, xacro)
@@ -14,3 +14,6 @@
         <color rgba= "0 0 0 1"/>
     </material>
+        <material name="red">
+        <color rgba= "1 0 0 1"/>
+    </material>
 </robot>

File: description/robot.urdf.xacro (robot description, xacro)
@@ -5,5 +5,6 @@
     <xacro:include filename="inertial_macro.xacro"/>
     <xacro:include filename="robot_core.xacro"/>
-    <xacro:include filename="gazebo_control.xacro"/>
+    <!--xacro:include filename="gazebo_control.xacro"-->
+    <xacro:include filename="ros2_control.xacro"/>
     <xacro:include filename="lidar.xacro"/>
 </robot>
