Commit message: SLAM

File: description/robot_core.xacro (robot description, xacro)
@@ -8,4 +8,11 @@
         <origin xyz="-0.1 0 0"/>
     </joint>
+    <joint name="base_footprint_joint" type="fixed">
+        <parent link="base_link"/>
+        <child link="base_footprint"/>
+        <origin xyz="0 0 -0.025"/>
+    </joint>
+    <link name="base_footprint">
+    </link>
     <!-- chassis link -->
     <link name="chassis">

Commit message: update ros2_control

File: description/robot_core.xacro (robot description, xacro)
@@ -54,5 +54,5 @@
         <collision>
             <geometry>
-                <cylinder radius="0.05" length="0.04"/>
+                <sphere radius="0.05"/>
             </geometry>
         </collision>
@@ -81,5 +81,5 @@
         <collision>
             <geometry>
-                <cylinder radius="0.05" length="0.04"/>
+                <sphere radius="0.05" />
             </geometry>
         </collision>
